Commit message: update mapping and remove velodyne

File: src/nexus_4wd_mecanum_description/urdf/nexus_4wd_mecanum.xacro (robot description, xacro)
@@ -407,52 +407,4 @@
     </visual>
   </link>
-  <joint name="velodyne_base_mount_joint" type="fixed">
-      <!-- <xacro:insert_block name="origin" />  -->
-      <parent link="base_link"/>
-      <child link="velodyne_base_link"/>
-  </joint>
-  <link name="velodyne_base_link">
-      <inertial>
-        <mass value="0.83"/>
-        <origin xyz="0 0 0.03585"/>
-        <inertia ixx="${(0.83 * (3.0*0.0516*0.0516 + 0.0717*0.0717)) / 12.0}" ixy="0" ixz="0"
-          iyy="${(0.83 * (3.0*0.0516*0.0516 + 0.0717*0.0717)) / 12.0}" iyz="0"
-          izz="${0.5 * 0.83 * (0.0516*0.0516)}"/>
-      </inertial>
-      <visual>
-        <geometry>
-          <mesh filename="package://velodyne_description/meshes/VLP16_base_1.dae" />
-        </geometry>
-      </visual>
-      <visual>
-        <geometry>
-          <mesh filename="package://velodyne_description/meshes/VLP16_base_2.dae" />
-        </geometry>
-      </visual>
-      <collision>
-        <origin rpy="0 0 0" xyz="0 0 0.03585"/>
-        <geometry>
-          <cylinder radius="0.0516" length="0.0717"/>
-        </geometry>
-      </collision>
-  </link>
-  <joint name="velodyne_base_scan_joint" type="fixed" >
-      <origin xyz="0 0 0.0377" rpy="0 0 0" />
-      <parent link="velodyne_base_link" />
-      <child link="velodyne"/>
-  </joint>
-  <link name="velodyne">
-      <inertial>
-        <mass value="0.01"/>
-        <origin xyz="0 0 0"/>
-        <inertia ixx="1e-7" ixy="0" ixz="0" iyy="1e-7" iyz="0" izz="1e-7"/>
-      </inertial>
-      <visual>
-        <origin xyz="0 0 -0.0377" />
-        <geometry>
-          <mesh filename="package://velodyne_description/meshes/VLP16_scan.dae" />
-        </geometry>
-      </visual>
-  </link>
   <!-- Include controller plugin for Gazebo -->
   <xacro:include filename="$(find nexus_4wd_mecanum_description)/urdf/nexus_4wd_mecanum.gazebo" />

Commit message: updatte multi waypoint planner

File: src/nexus_4wd_mecanum_description/urdf/nexus_4wd_mecanum.xacro (robot description, xacro)
@@ -39,5 +39,5 @@
   </link>
   <joint name="upper_left_wheel_shaft_joint" type="fixed">
-    <origin xyz="0.150 0.108 0.0" rpy="0 0 0" />
+    <origin xyz="0.150 0.108 0.0" rpy="0 0 0"/>
     <parent link="base_link"/>
     <child link="upper_left_wheel_shaft" />
@@ -50,4 +50,9 @@
     <child link="camera_link"/>
   </joint>
+  <joint name="imu_joint" type="fixed">
+    <origin xyz="0.0 0.0 0.3" rpy="0 0 0"/>
+    <parent link="base_link"/>
+    <child link="imu_link"/>
+  </joint>
   <joint name="depth_joint" type="fixed">
     <axis xyz="0 1 0" />
@@ -70,4 +75,24 @@
       </geometry>
       <material name="red"/>
+    </visual>
+    <inertial>
+      <mass value="1e-5" />
+      <origin xyz="0 0 0" rpy="0 0 0"/>
+      <inertia ixx="1e-6" ixy="0" ixz="0" iyy="1e-6" iyz="0" izz="1e-6" />
+    </inertial>
+  </link>
+  <link name="imu_link">
+    <collision>
+      <origin xyz="0 0 0" rpy="0 0 0"/>
+      <geometry>
+    <box size="${camera_link} ${camera_link} ${camera_link}"/>
+      </geometry>
+    </collision>
+    <visual>
+      <origin xyz="0 0 0" rpy="0 0 0"/>
+      <geometry>
+    <box size="${camera_link} ${camera_link} ${camera_link}"/>
+      </geometry>
+      <!-- <material name="red"/> -->
     </visual>
     <inertial>
@@ -438,5 +463,5 @@
   </link>
   <joint name="velodyne_base_scan_joint" type="fixed" >
-      <origin xyz="0 0 0.0377" rpy="0 0 0" />
+      <origin xyz="0 0 0.08" rpy="0 0 0" />
       <parent link="velodyne_base_link" />
       <child link="velodyne"/>
